File: Schematics/MCU.kicad_sch (KiCad schematic)
At the start: 4 parts, among them U1 ATmega64A-A, Y1 16MHz

Commit message: PCB
Connections:
- net ServoPWM2: now reaches U1.17 (PB7)
- net ServoPWM1: now reaches U1.32 (PD7)
- net ServoPWM: no longer names the net of U1.51 (PA0)
- no-connect marks 36 -> 35
Changed lines of the file:
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@@
   (junction (at 125.73 66.04) (diameter 0) (color 0 0 0 0)
   )
+  (no_connect (at 162.56 60.96))
+  (no_connect (at 132.08 147.32))
   (no_connect (at 132.08 96.52))
   (no_connect (at 132.08 93.98))
@@
   (no_connect (at 162.56 142.24))
   (no_connect (at 162.56 144.78))
-  (no_connect (at 162.56 147.32))
-  (no_connect (at 132.08 147.32))
   (no_connect (at 132.08 144.78))
   (no_connect (at 132.08 142.24))
@@
   (no_connect (at 162.56 96.52))
   (no_connect (at 162.56 99.06))
-  (no_connect (at 162.56 101.6))
   (no_connect (at 162.56 106.68))
   (no_connect (at 162.56 109.22))
@@
     (stroke (width 0) (type default) (color 0 0 0 0))
   )
+  (wire (pts (xy 162.56 147.32) (xy 174.625 147.32))
+    (stroke (width 0) (type default) (color 0 0 0 0))
+  )
   (wire (pts (xy 149.86 53.34) (xy 149.86 45.72))
     (stroke (width 0) (type default) (color 0 0 0 0))
@@
     (stroke (width 0) (type default) (color 0 0 0 0))
   )
-  (wire (pts (xy 162.56 60.96) (xy 174.625 60.96))
-    (stroke (width 0) (type default) (color 0 0 0 0))
-  )
   (wire (pts (xy 162.56 129.54) (xy 174.625 129.54))
     (stroke (width 0) (type default) (color 0 0 0 0))
@@
     (stroke (width 0) (type default) (color 0 0 0 0))
   )
+  (wire (pts (xy 162.56 101.6) (xy 174.625 101.6))
+    (stroke (width 0) (type default) (color 0 0 0 0))
+  )
   (wire (pts (xy 118.11 116.84) (xy 132.08 116.84))
     (stroke (width 0) (type default) (color 0 0 0 0))
@@
     )
   )
-  (global_label "ServoPWM" (shape input) (at 174.625 60.96 0) (fields_autoplaced)
-    (effects (font (size 1.27 1.27)) (justify left))
-    (property "Intersheet References" "${INTERSHEET_REFS}" (id 0) (at 186.4119 60.8806 0)
+  (global_label "ServoPWM2" (shape input) (at 174.625 101.6 0) (fields_autoplaced)
+    (effects (font (size 1.27 1.27)) (justify left))
+    (property "Intersheet References" "${INTERSHEET_REFS}" (id 0) (at 187.6214 101.6794 0)
       (effects (font (size 1.27 1.27)) (justify left) hide)
     )
@@
     (effects (font (size 1.27 1.27)) (justify left))
     (property "Intersheet References" "${INTERSHEET_REFS}" (id 0) (at 181.6343 91.3606 0)
+      (effects (font (size 1.27 1.27)) (justify left) hide)
+    )
+  )
+  (global_label "ServoPWM1" (shape input) (at 174.625 147.32 0) (fields_autoplaced)
+    (effects (font (size 1.27 1.27)) (justify left))
+    (property "Intersheet References" "${INTERSHEET_REFS}" (id 0) (at 187.6214 147.2406 0)
       (effects (font (size 1.27 1.27)) (justify left) hide)
     )
@@
     (pin "1")
     (pin "2")
+  )
+  (symbol (lib_id "power:VCC") (at 129.54 76.2 0) (unit 1)
+    (in_bom yes) (on_board yes)
+    (property "Reference" "#PWR0101" (id 0) (at 129.54 80.01 0)
+      (effects (font (size 1.27 1.27)) hide)
+    )
+    (property "Value" "VCC" (id 1) (at 131.445 77.47 0)
+      (effects (font (size 1.27 1.27)) (justify right))
+    )
+    (property "Footprint" "" (id 2) (at 129.54 76.2 0)
+      (effects (font (size 1.27 1.27)) hide)
+    )
+    (property "Datasheet" "" (id 3) (at 129.54 76.2 0)
+      (effects (font (size 1.27 1.27)) hide)
+    )
+    (pin "1")
   )
   (symbol (lib_id "power:Earth") (at 107.95 76.2 0) (unit 1)
@@
     (pin "9")
   )
-  (symbol (lib_id "power:VCC") (at 129.54 76.2 90) (unit 1)
-    (in_bom yes) (on_board yes) (fields_autoplaced)
-    (property "Reference" "#PWR03" (id 0) (at 133.35 76.2 0)
-      (effects (font (size 1.27 1.27)) hide)
-    )
-    (property "Value" "VCC" (id 1) (at 124.46 76.2 0))
-    (property "Footprint" "" (id 2) (at 129.54 76.2 0)
-      (effects (font (size 1.27 1.27)) hide)
-    )
-    (property "Datasheet" "" (id 3) (at 129.54 76.2 0)
-      (effects (font (size 1.27 1.27)) hide)
-    )
-    (pin "1")
-  )
   (symbol (lib_id "Device:C_Small") (at 116.84 71.12 90) (unit 1)
