File: Smart Floor Register.kicad_pcb (KiCad board)
At the start: 2 copper layers, 115.9 x 79.2 mm, 68 parts, among them J1 Fan 1, J2 Fan 2, J3 USB_B_Micro, J4 AVR-ISP-6, M1 Motor_Servo, SW1 RESET, SW2 PEN, SW3 Fan, SW4 Servo, U1 ATmega64A-A, U2 AD8539ARMZ-REEL, U3 AD8539ARMZ-REEL, U4 LTC1695, U5 LTC1695, U6 XC9142B50CMR-G, Y1 16MHz

Commit message: PCB
Parts:
- removed BT1: 18650, SFRFootprints:1049P
- moved M1 96.2 mm to (110.1, 93.6), turned to -90 degrees
- moved C3 81.0 mm to (110.5, 91.2), turned to 180 degrees
- moved L1 78.6 mm to (138.7, 72.9), turned to 90 degrees
- moved J1 77.9 mm to (109.9, 88.5), turned to -90 degrees
- moved C5 77.8 mm to (144.3, 72.9), turned to -90 degrees
- moved U6 76.2 mm to (141.5, 72.9), turned to 90 degrees
- moved BT2 74.5 mm to (114.2, 71.5), turned to -90 degrees
- moved U4 71.3 mm to (110.4, 88.6), turned to 180 degrees
- moved C4 51.3 mm to (137.2, 86.1)
- moved U5 43.8 mm to (137.2, 88.6)
- moved R20 37.8 mm to (103.6, 141.2)
- moved S1 37.6 mm to (104.9, 69.8)
- moved A4 36.9 mm to (147.0, 100.8)
- moved J2 35.5 mm to (147.0, 88.5), turned to -90 degrees
- moved SW4 34.5 mm to (103.6, 144.3)
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Connections:
- U1 pad 54: Thermistor -> ThermistorB
- U1 pad 55: ThermistorA -> ThermopileB
- U1 pad 56: ThermopileC -> ThermopileA
- U1 pad 57: ThermistorD -> Thermistor
- U1 pad 59: ThermistorC -> ThermopileC
- U1 pad 60: ThermopileB -> ThermistorC
- U1 pad 61: ThermopileA -> ThermistorD
Routing:
- net VCC: track 0.00 -> 190.4 mm, vias 0 -> 7
- net Shifted Ground: track 0.00 -> 74.8 mm
- net +5V: track 0.00 -> 61.1 mm, vias 0 -> 3
- net MOSI: track 0.00 -> 51.8 mm, vias 0 -> 1
- net SCK: track 0.00 -> 50.0 mm, vias 0 -> 1
- net MISO: track 0.00 -> 49.5 mm, vias 0 -> 1
- net SDA: track 0.00 -> 38.2 mm, vias 0 -> 3
- net SCL: track 0.00 -> 33.8 mm, vias 0 -> 3
- net MotorEnable: track 0.00 -> 30.4 mm
- net Net-(A4-Pad2): track 0.00 -> 28.5 mm, vias 0 -> 2
- net Net-(A1-Pad2): track 0.00 -> 28.2 mm, vias 0 -> 2
- net ThermistorB: track 0.00 -> 27.9 mm, vias 0 -> 2
- net ThermistorC: track 0.00 -> 26.6 mm, vias 0 -> 2
- net ThermistorD: track 0.00 -> 24.7 mm, vias 0 -> 2
- net ServoPWM: track 0.00 -> 23.0 mm, vias 0 -> 2
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- added copper zone on B.Cu, net Earth
- added copper zone on F.Cu, net Earth
Other:
- board size 115.9 x 79.2 mm -> 46.8 x 79.1 mm

Commit message: PCB
Parts:
- moved TP11 90.9 mm to (137.7, 132.3)
- moved TP8 87.1 mm to (141.2, 132.3)
- moved TP9 78.8 mm to (135.9, 95.8)
- moved TP10 77.6 mm to (137.9, 101.3)
- moved TP14 74.6 mm to (125.0, 128.7)
- moved TP16 71.2 mm to (110.7, 130.0)
- moved TP12 71.2 mm to (137.9, 107.2)
- moved TP6 70.9 mm to (134.9, 74.8)
- moved TP13 69.0 mm to (115.5, 126.2)
- moved TP2 68.6 mm to (127.5, 116.3)
- moved TP15 62.8 mm to (106.7, 130.0)
- moved TP1 54.1 mm to (111.8, 84.3)
- moved TP4 52.9 mm to (109.5, 101.3)
- moved TP3 51.6 mm to (109.0, 84.3)
- moved TP7 51.0 mm to (112.5, 95.5)
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Connections:
- BT2 pad 3: (no net) -> Earth
- BT2 pad 4: (no net) -> Net-(BT1-Pad1)
- U1 pad 49: FanActivate -> ServoActivate
- U1 pad 50: ServoActivate -> FanActivate
Routing:
- net Net-(BT1-Pad1): track 12.7 -> 111.9 mm, vias 0 -> 2
- net VCC: track 190.4 -> 263.2 mm, vias 7 -> 9
- net Earth: track 20.4 -> 92.9 mm, vias 2 -> 13
- net ~{RESET}: track 0.00 -> 62.9 mm, vias 0 -> 2
- net ServoActivate: track 0.00 -> 46.3 mm, vias 0 -> 2
- net ~{PEN}: track 0.00 -> 46.1 mm, vias 0 -> 2
- net FanActivate: track 0.00 -> 45.1 mm, vias 0 -> 2
- net Shifted Ground: track 74.8 -> 119.2 mm, vias 0 -> 2
- net ThermopileD: track 18.4 -> 37.1 mm, vias 0 -> 2
- net ThermopileC: track 18.6 -> 36.2 mm, vias 0 -> 2
- net ThermopileA: track 18.4 -> 35.5 mm, vias 0 -> 2
- net ThermopileB: track 19.3 -> 34.3 mm, vias 0 -> 2
- net +5V: track 61.1 -> 71.5 mm
- net MotorEnable: track 30.4 -> 33.6 mm
- net ThermistorD: track 24.7 -> 27.7 mm
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
Commit message: PCB
Parts:
- added M2: Motor_Servo, SFRFootprints:Servo, F.Cu at (135.4, 86.9)
- added TP17: TestPoint, TestPoint:TestPoint_Pad_D1.5mm, F.Cu at (131.4, 80.8)
- SW1: value RESET -> Rest
- moved TP9 18.6 mm to (137.3, 77.2)
- moved TP8 12.3 mm to (139.2, 120.2)
- moved U4 9.91 mm to (110.4, 98.6)
- moved C3 9.91 mm to (110.5, 101.1)
- moved TP1 9.91 mm to (111.8, 94.2)
- moved TP3 9.91 mm to (109.0, 94.2)
- moved TP13 9.63 mm to (114.2, 135.8)
- moved C4 9.40 mm to (137.2, 95.5)
- moved U5 9.40 mm to (137.2, 98.0)
- moved TP16 8.75 mm to (119.2, 127.8)
- moved TP11 8.56 mm to (129.8, 135.7)
- moved J1 8.14 mm to (109.9, 96.6)
- moved TP6 7.86 mm to (142.4, 77.2)
- moved J2 7.75 mm to (147.0, 96.2)
- moved A2 7.26 mm to (109.4, 113.8)
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Connections:
- M1 pad 1: ServoPWM -> ServoPWM1
- SW1 pad 2: ~{RESET} -> Earth
- SW2 pad 2: ~{PEN} -> Earth
- TP7 pad 1: ServoPWM -> ServoPWM1
- U1 pad 17: unconnected-(U1-Pad17) -> ServoPWM2
- U1 pad 32: unconnected-(U1-Pad32) -> ServoPWM1
- U1 pad 51: ServoPWM -> unconnected-(U1-Pad51)
Routing:
- net Earth: track 92.9 -> 161.4 mm, vias 13 -> 16
- net ServoPWM: track 25.9 -> 0.00 mm, vias 3 -> 0
- net Shifted Ground: track 119.2 -> 98.1 mm, vias 2 -> 8
- net ServoPWM2: track 0.00 -> 16.2 mm
- net +5V: track 71.5 -> 80.5 mm, vias 3 -> 5
- net ServoPWM1: track 0.00 -> 8.65 mm
- net ThermopileA: track 35.5 -> 27.9 mm
- net SCL: track 36.4 -> 30.8 mm
- net ServoActivate: track 46.3 -> 40.8 mm, vias 2 -> 0
- net SCK: track 49.8 -> 44.8 mm
- net FanActivate: track 45.1 -> 40.3 mm, vias 2 -> 0
- net ~{PEN}: track 46.1 -> 41.3 mm
- net MOSI: track 53.5 -> 48.8 mm
- net ThermopileC: track 36.2 -> 31.8 mm
- net Net-(A4-Pad2): track 28.5 -> 32.2 mm
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
Commit message: Updated Gerbers
Connections:
- SW1 pad 1: Earth -> ~{RESET}
- SW2 pad 2: Earth -> ~{PEN}
Routing:
- net ~{PEN}: track 41.3 -> 45.5 mm
- net ~{RESET}: track 62.8 -> 67.0 mm
Changed lines of the file:
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@@
       (outputformat 1)
       (mirror false)
-      (drillshape 1)
+      (drillshape 0)
       (scaleselection 1)
-      (outputdirectory "")
+      (outputdirectory "Gerbers/")
     )
   )
@@
     (fp_line (start -1.6 -0.8) (end 1.6 -0.8) (layer "F.Fab") (width 0.1))
     (fp_line (start -1.6 0.8) (end -1.6 -0.8) (layer "F.Fab") (width 0.1))
-    (pad "1" smd roundrect (at -1.55 0) (size 1.3 1.75) (layers "F.Cu" "F.Paste" "F.Mask") (roundrect_rratio 0.192308)
+    (pad "1" smd roundrect (at -1.55 0) (size 1.3 1.75) (layers "F.Cu" "F.Paste" "F.Mask") (roundrect_rratio 0.1923076923)
       (net 15 "VCC") (pintype "passive"))
-    (pad "2" smd roundrect (at 1.55 0) (size 1.3 1.75) (layers "F.Cu" "F.Paste" "F.Mask") (roundrect_rratio 0.192308)
+    (pad "2" smd roundrect (at 1.55 0) (size 1.3 1.75) (layers "F.Cu" "F.Paste" "F.Mask") (roundrect_rratio 0.1923076923)
       (net 32 "Thermistor") (pintype "passive"))
     (model "${KICAD6_3DMODEL_DIR}/Resistor_SMD.3dshapes/R_1206_3216Metric.wrl"
@@
       (net 1 "Earth") (pinfunction "A") (pintype "passive"))
     (pad "2" smd rect (at 1.849999 -0.750001) (size 0.508 0.889) (layers "F.Cu" "F.Paste" "F.Mask")
-      (net 1 "Earth") (pinfunction "A") (pintype "passive"))
+      (net 37 "~{PEN}") (pinfunction "A") (pintype "passive"))
     (pad "2" smd rect (at 1.849999 0.750001) (size 0.508 0.889) (layers "F.Cu" "F.Paste" "F.Mask")
-      (net 1 "Earth") (pinfunction "A") (pintype "passive"))
+      (net 37 "~{PEN}") (pinfunction "A") (pintype "passive"))
   )
   (footprint "SFRFootprints:R-667843" (layer "F.Cu")
@@
     (fp_circle (center -1.85 -2.655) (end -1.469 -2.655) (layer "F.Fab") (width 0.1) (fill none))
     (pad "1" smd rect (at -1.849999 0.750001) (size 0.508 0.889) (layers "F.Cu" "F.Paste" "F.Mask")
-      (net 1 "Earth") (pinfunction "A") (pintype "passive"))
+      (net 25 "~{RESET}") (pinfunction "A") (pintype "passive"))
     (pad "1" smd rect (at -1.849999 -0.750001) (size 0.508 0.889) (layers "F.Cu" "F.Paste" "F.Mask")
-      (net 1 "Earth") (pinfunction "A") (pintype "passive"))
+      (net 25 "~{RESET}") (pinfunction "A") (pintype "passive"))
     (pad "2" smd rect (at 1.849999 -0.750001) (size 0.508 0.889) (layers "F.Cu" "F.Paste" "F.Mask")
       (net 1 "Earth") (pinfunction "A") (pintype "passive"))
@@
   (segment (start 127.876998 143.903002) (end 126.746 145.034) (width 0.25) (layer "B.Cu") (net 24))
   (segment (start 130.556 141.224) (end 136.52975 141.224) (width 0.25) (layer "F.Cu") (net 25))
+  (segment (start 135.614801 145.022001) (end 135.614801 143.521999) (width 0.25) (layer "F.Cu") (net 25))
   (segment (start 127.171 95.678) (end 127.171 97.381197) (width 0.25) (layer "F.Cu") (net 25))
   (segment (start 127.171 97.381197) (end 127.389903 97.6001) (width 0.25) (layer "F.Cu") (net 25))
+  (segment (start 135.614801 143.521999) (end 135.614801 142.138949) (width 0.25) (layer "F.Cu") (net 25))
+  (segment (start 135.614801 142.138949) (end 136.52975 141.224) (width 0.25) (layer "F.Cu") (net 25))
   (segment (start 129.286 142.494) (end 130.556 141.224) (width 0.25) (layer "F.Cu") (net 25))
   (via (at 127.389903 97.6001) (size 0.8) (drill 0.4) (layers "F.Cu" "B.Cu") (net 25))
@@
   (segment (start 125.563637 119.510889) (end 127.312348 121.2596) (width 0.25) (layer "B.Cu") (net 36))
   (segment (start 127.312348 121.2596) (end 130.6068 121.2596) (width 0.25) (layer "B.Cu") (net 36))
+  (segment (start 120.518799 143.471199) (end 120.518799 142.095299) (width 0.25) (layer "F.Cu") (net 37))
   (segment (start 119.5791 141.1224) (end 119.5625 141.139) (width 0.25) (layer "F.Cu") (net 37))
   (segment (start 131.271 109.378) (end 131.271 110.5954) (width 0.25) (layer "F.Cu") (net 37))
+  (segment (start 120.518799 142.095299) (end 119.5625 141.139) (width 0.25) (layer "F.Cu") (net 37))
   (segment (start 131.271 110.5954) (end 131.318 110.6424) (width 0.25) (layer "F.Cu") (net 37))
+  (segment (start 120.518799 144.971201) (end 120.518799 143.471199) (width 0.25) (layer "F.Cu") (net 37))
   (segment (start 120.904 141.1224) (end 119.5791 141.1224) (width 0.25) (layer "F.Cu") (net 37))
   (via (at 131.318 110.6424) (size 0.8) (drill 0.4) (layers "F.Cu" "B.Cu") (net 37))

Commit message: Finalized PCB
Parts:
- R13, R14, R2, R4: value 1k -> 100k
- SW1: value Rest -> R-667843_MIT
- SW2: value PEN -> R-667843_MIT
- SW3: value Fan -> R-667843_MIT
- SW4: value Servo -> R-667843_MIT
- U2, U3: value AD8539ARMZ-REEL -> Opamp_Dual
- U6: value XC9142B50CMR-G -> SC_50CMR-G_TOR
- moved TP8 27.2 mm to (118.2, 137.6)
- moved TP15 16.2 mm to (115.5, 137.6)
- moved TP16 11.6 mm to (112.9, 137.6)
- moved TP6 11.3 mm to (131.2, 75.3)
- moved R11 10.8 mm to (137.1, 124.6)
- moved R13 10.8 mm to (126.4, 122.8)
- moved SW2 10.0 mm to (108.7, 144.2), turned to 180 degrees
- moved SW3 9.99 mm to (118.6, 144.1)
- moved TP11 9.11 mm to (120.9, 137.6)
- moved TP13 7.76 mm to (108.3, 130.8)
- moved R5 5.49 mm to (126.4, 124.6)
- moved R12 5.19 mm to (121.3, 124.6)
- moved TP2 4.56 mm to (126.2, 114.2)
- moved TP9 2.21 mm to (135.1, 76.9)
- moved R4 1.78 mm to (121.3, 122.8), turned to 180 degrees
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Connections:
- A4 pad 1: Earth -> Shifted Ground
- A4 pad 2: Net-(A4-Pad2) -> ThermistorD
- A4 pad 3: ThermistorD -> Net-(A4-Pad3)
- A4 pad 4: Shifted Ground -> Earth
- R11 pad 1: ThermopileD -> Shifted Ground
- R11 pad 2: Shifted Ground -> Net-(R14-Pad1)
- R12 pad 1: Net-(R12-Pad1) -> Shifted Ground
- R12 pad 2: ThermopileD -> Net-(R4-Pad1)
- R14 pad 1: ThermopileC -> Net-(R14-Pad1)
- R14 pad 2: Shifted Ground -> ThermopileD
- R2 pad 1: ThermopileB -> ThermopileA
- R2 pad 2: Shifted Ground -> Net-(R3-Pad2)
- R3 pad 1: Net-(R3-Pad1) -> Shifted Ground
- R3 pad 2: ThermopileB -> Net-(R3-Pad2)
- R4 pad 2: ThermopileA -> ThermopileB
- R5 pad 1: ThermopileA -> Shifted Ground
- R5 pad 2: Shifted Ground -> Net-(R13-Pad1)
- R8 pad 1: VCC -> Thermistor
- R8 pad 2: Thermistor -> Earth
- R9 pad 1: Thermistor -> VCC
- R9 pad 2: Earth -> Thermistor
- U1 pad 55: ThermopileB -> ThermopileA
- U1 pad 56: ThermopileA -> ThermopileB
- U1 pad 58: ThermopileD -> ThermopileC
- U1 pad 59: ThermopileC -> ThermopileD
- U2 pad 1: ThermopileB -> ThermopileA
- U2 pad 2: Net-(R3-Pad1) -> Net-(R3-Pad2)
- U2 pad 3: Net-(A2-Pad2) -> Net-(A1-Pad2)
- U2 pad 5: Net-(A1-Pad2) -> Net-(A2-Pad2)
- U2 pad 7: ThermopileA -> ThermopileB
- U3 pad 1: ThermopileD -> ThermopileC
- U3 pad 2: Net-(R12-Pad1) -> Net-(R13-Pad1)
- U3 pad 3: Net-(A4-Pad2) -> Net-(A3-Pad2)
- U3 pad 5: Net-(A3-Pad2) -> Net-(A4-Pad3)
- U3 pad 6: Net-(R13-Pad1) -> Net-(R14-Pad1)
- U3 pad 7: ThermopileC -> ThermopileD
Routing:
- net Earth: track 161.4 -> 53.0 mm, vias 16 -> 18
- net Net-(A4-Pad2): track 32.2 -> 0.00 mm, vias 2 -> 0
- net Net-(A4-Pad3): track 0.00 -> 28.2 mm, vias 0 -> 2
- net VCC: track 262.2 -> 242.4 mm, vias 3 -> 7
- net ThermopileA: track 27.9 -> 46.3 mm, vias 2 -> 3
- net +5V: track 80.5 -> 93.7 mm, vias 5 -> 4
- net ThermopileC: track 31.8 -> 44.2 mm, vias 2 -> 3
- net ThermopileD: track 39.0 -> 49.0 mm, vias 4 -> 3
- net Net-(A3-Pad2): track 21.0 -> 28.3 mm
- net ThermopileB: track 34.9 -> 41.6 mm, vias 2 -> 3
- net ThermistorC: track 27.8 -> 34.0 mm
- net ThermistorB: track 27.5 -> 33.2 mm, vias 3 -> 2
- net ServoPWM2: track 16.2 -> 21.7 mm
- net Net-(R3-Pad2): track 0.00 -> 5.28 mm
- net Net-(R14-Pad1): track 0.00 -> 4.99 mm
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